File: esp8266-event-notifier.sch (EAGLE design)
At the start: 10 parts, among them U1 SN74HC595N, U2 SN74HC595N, U3 SN74HC595N, U4 SN74HC595N

Commit message: test-diplsay
Parts:
- added R10, R11, R12, R13, R14, R15, R16, R17, R18, R19, R20, R21, R22, R23, R24, R25, R26, R27, R28, R29, R30, R31, R32, R33, R34, R35, R36, R5, R6, R7, R8, R9: 330, adafruit:R-US_R0805
Connections:
- removed net N$21 (its old number): U3.QF
- removed net N$27 (its old number): U3.QA
- removed net N$28: U4.QH
- removed net N$29 (its old number): U4.QG
- new net N$13: R8.2, U1.QE
- new net N$22: R16.1
- new net N$31: R14.2, U2.QG
- new net N$37: R20.2, U2.QA
- new net N$38: R21.1
- new net N$39: R22.1
- new net N$50: R23.1
- new net N$52: R24.1
- new net N$53: R25.1
- new net N$54: R26.1
- new net N$55: R27.1
- new net N$56: R28.1
- new net N$60: R21.2, U3.QH
- new net N$61: R22.2, U3.QG
- new net N$62: R23.2, U3.QF
- new net N$63: R24.2, U3.QE
- new net N$64: R25.2, U3.QD
- new net N$65: R26.2, U3.QC
- new net N$66: R27.2, U3.QB
- new net N$67: R28.2, U3.QA
- new net N$68: R29.1
- new net N$69: R30.1
- new net N$70: R31.1
- new net N$72: R32.1
- new net N$73: R33.1
- new net N$74: R34.1
- new net N$75: R35.1
- new net N$76: R36.1
- new net N$80: R29.2, U4.QH
- new net N$81: R30.2, U4.QG
- new net N$82: R31.2, U4.QF
- new net N$83: R32.2, U4.QE
- new net N$84: R33.2, U4.QD
- new net N$85: R34.2, U4.QC
- new net N$86: R35.2, U4.QB
- new net N$87: R36.2, U4.QA
- new net VCC: U$1.3V@1, U1.SCL, U2.SCL, U3.SCL, U4.SCL
- net GND: no longer U1.SCL, U2.SCL, U3.SCL, U4.SCL
- net N$1: now also R5.1; no longer U1.QH
- net N$10: now also R5.2, U1.QH; no longer U2.QH
- net N$11: now also R6.2, U1.QG; no longer U2.QG
- net N$12: now also R7.2, U1.QF; no longer U2.QF
- net N$14: now also R9.2, U1.QD; no longer U2.QE
- net N$15: now also R10.2, U1.QC; no longer U2.QD
- net N$16: now also R11.2, U1.QB; no longer U2.QC
- net N$17: now also R12.2, U1.QA; no longer U2.QB
- net N$18: now also R13.1; no longer U2.QA
- net N$19: now also R14.1; no longer U3.QH
- net N$2: now also R6.1; no longer U1.QG
- net N$20: now also R15.1; no longer U3.QG
- net N$23: now also R17.1; no longer U3.QE
- net N$24: now also R18.1; no longer U3.QD
- net N$25: now also R19.1; no longer U3.QC
- net N$26: now also R20.1; no longer U3.QB
- net N$3: now also R7.1; no longer U1.QF
- net N$30: now also R13.2, U2.QH; no longer U4.QF
- net N$32: now also R15.2, U2.QF; no longer U4.QE
- net N$33: now also R16.2, U2.QE; no longer U4.QD
- net N$34: now also R17.2, U2.QD; no longer U4.QC
- net N$35: now also R18.2, U2.QC; no longer U4.QB
- net N$36: now also R19.2, U2.QB; no longer U4.QA
- net N$5: now also R8.1; no longer U1.QE
- net N$6: now also R9.1; no longer U1.QD
- net N$7: now also R10.1; no longer U1.QC
- net N$8: now also R11.1; no longer U1.QB
- net N$9: now also R12.1; no longer U1.QA
Other:
- moved on the sheet: U2, U3, U4

Commit message: WORKING!!!
seven segment display - working
led - working
calendar event detection - working
To Do: set it to check for events earlier if it detects one is coming soon
Connections:
- removed net N$57 (its old number): U2.QH*, U3.SER
- removed net N$77 (its old number): U3.QH*, U4.SER
- new net N$38: U2.RCK
- new net N$39: U2.SCK
- new net N$42: U1.QH*
- new net N$50: U2.QH*
- new net N$60: U3.SER
- new net N$69: U3.RCK
- new net N$70: U3.SCK
- new net N$72: U3.QH*
- new net N$83: U4.SER
- new net N$92: U4.RCK
- new net N$93: U4.SCK
- new net N$95: U4.QH*
- net N$27: no longer U1.QH*
- net N$29: no longer U2.RCK, U3.RCK, U4.RCK
- net N$78: no longer U2.SCK, U3.SCK, U4.SCK
Other:
- moved on the sheet: U3, U4

Commit message: Update esp8266-event-notifier.sch
Parts:
- added CN1: 9V, adafruit:DCBARRELPTH
Connections:
- net N$40 renamed SER
- removed net N$39: U2.SCK
- removed net N$42: U1.QH*
- removed net N$60: U3.SER
- removed net N$69: U3.RCK
- removed net N$70: U3.SCK
- removed net N$78: U$1.D6, U1.SCK
- removed net N$83: U4.SER
- removed net N$92: U4.RCK
- removed net N$93: U4.SCK
- removed net N$95: U4.QH*
- new net CLK: U$1.D6, U1.SCK, U2.SCK, U3.SCK, U4.SCK
- new net LATCH: U$1.D7, U1.RCK, U2.RCK, U3.RCK, U4.RCK
- net N$27: now also U1.QH*
- net N$29: now also CN1.PWR, U$1.VIN; no longer U$1.D7, U1.RCK
- net N$38: now also CN1.GND, U$1.GND@2; no longer U2.RCK
- net N$50: now also U3.SER
- net N$72: now also U4.SER
