File: esp8266_event_notifier_schematic.sch (EAGLE design)
At the start: 43 parts, among them CN1 9V, U1 SN74HC595N, U2 SN74HC595N, U3 SN74HC595N, U4 SN74HC595N

Commit message: Added schematic pdf
Also removed library files, the user should copy them directly from the source
Other:
- note added: "By: Bryce Dombrowski https://www.brycedombrowski.com"
- note added: "ESP8266 Event Notifier"
- moved on the sheet: U1, U2, U3, U4
